File: m1/hardware/OpenChordM1/OpenChordM1.kicad_sch (KiCad schematic)
At the start: 74 parts, among them J1 USB4105-GF-A, J2 SJ1-3523N (OUT), J3 SJ1-3523N (IN), SW1 SW_Gateron_LP, SW10 EVQ-PUA02K, SW11 EVQ-PUA02K, SW13 TS-1187A-B-A-B, SW2 SW_Gateron_LP, SW3 SW_Gateron_LP, SW4 SW_Gateron_LP, SW5 SW_Gateron_LP, SW6 SW_Gateron_LP, SW7 SW_Gateron_LP, SW8 SW_Gateron_LP, SW9 EVQ-PUA02K, U1 RP2040, U2 CT_Slider_Chev_3_74d5_15_noESD, U3 IQS572-BL-QNR, U4 AT42QT2120-XUR, U5 CT_Trackpad_7x7_37D75, U6 W25Q16JVSSIQ, U7 AP2112K-3.3TRG1, U8 USBLC6-2SC6, U9 TLP2361, Y1 ABM8-272-T3

Commit message: Lock rev A to in-stock parts and sync the board docs.
Use EVQPUC02K side buttons and W25Q32JVSSIQ flash, and add the Hroparts USB-C library so J1 can leave the out-of-stock GCT connector.
Parts:
- removed J1: USB4105-GF-A, oc-usb:USB4105-GF-A, symbol oc-usb:USB4105-GF-A
- added J4: TYPE-C-31-M-12, oc-usb:TYPE-C-31-M-12, symbol oc-usb:TYPE-C-31-M-12
- added R30: 10k, Resistor_SMD:R_0603_1608Metric, symbol Device:R
- C1, C14, C3, C4, C5, C6: LCSC Part (none) -> C14663; MPN (none) -> CC0603KRX7R9BB104; Manufacturer (none) -> YAGEO
- C10, C11: LCSC Part (none) -> C1713; MPN (none) -> CL21A106KOQNNNE; Manufacturer (none) -> Samsung
- C12, C13: LCSC Part (none) -> C1644; MPN (none) -> CL10C150JB8NNNC; Manufacturer (none) -> Samsung
- C2: value 100nF -> 1uF; LCSC Part (none) -> C14664; MPN (none) -> CC0603KRX5R8BB105; Manufacturer (none) -> YAGEO
- C7, C8, C9: LCSC Part (none) -> C14664; MPN (none) -> CC0603KRX5R8BB105; Manufacturer (none) -> YAGEO
- D1: LCSC Part (none) -> C2128; MPN (none) -> 1N4148WS; Manufacturer (none) -> JSCJ
- DS1: MPN (none) -> SSD1306 0.91in 4-pin; Manufacturer (none) -> generic
- R1, R2: LCSC Part (none) -> C23186; MPN (none) -> 0603WAF5101T5E; Manufacturer (none) -> UNI-ROYAL
- R10: LCSC Part (none) -> C22962; MPN (none) -> 0603WAF2200T5E; Manufacturer (none) -> UNI-ROYAL
- R11: LCSC Part (none) -> C22859; MPN (none) -> 0603WAF100JT5E; Manufacturer (none) -> UNI-ROYAL
- R12: LCSC Part (none) -> C23140; MPN (none) -> 0603WAF330JT5E; Manufacturer (none) -> UNI-ROYAL
- R13, R14, R15, R6: LCSC Part (none) -> C98220; MPN (none) -> RC0603FR-0710KL; Manufacturer (none) -> YAGEO
- R16, R17, R18, R19, R20, R21, R22, R23, R24, R25, R26, R27, R28, R29, R5, R7: LCSC Part (none) -> C21190; MPN (none) -> 0603WAF1001T5E; Manufacturer (none) -> UNI-ROYAL
- R3, R4: LCSC Part (none) -> C23345; MPN (none) -> 0603WAF220JT5E; Manufacturer (none) -> UNI-ROYAL
- R8, R9: LCSC Part (none) -> C23162; MPN (none) -> 0603WAF4701T5E; Manufacturer (none) -> UNI-ROYAL
- SW1, SW2, SW3, SW4, SW5, SW6, SW7, SW8: MPN (none) -> KS-33 hotswap socket; Manufacturer (none) -> Gateron
- SW10, SW11, SW9: value EVQ-PUA02K -> EVQPUC02K; footprint oc-btn:EVQ-PUA02K -> oc-btn:EVQPUC02K; symbol oc-btn:EVQ-PUA02K -> oc-btn:EVQPUC02K; LCSC Part C128539 -> C79174; MPN EVQ-PUA02K -> EVQPUC02K
- U1: LCSC Part (none) -> C2040; MPN (none) -> RP2040; Manufacturer (none) -> Raspberry Pi
- U4: Manufacturer MICROCHIP(美国微芯) -> Microchip
- U6: value W25Q16JVSSIQ -> W25Q32JVSSIQ; LCSC Part (none) -> C179173; MPN (none) -> W25Q32JVSSIQ; Manufacturer (none) -> Winbond
- U7: LCSC Part (none) -> C51118; MPN (none) -> AP2112K-3.3TRG1; Manufacturer (none) -> Diodes Incorporated
- U8: LCSC Part (none) -> C7519; MPN (none) -> USBLC6-2SC6; Manufacturer (none) -> ST
- U9: LCSC Part (none) -> C107626; MPN (none) -> TLP2361(TPL,E); Manufacturer (none) -> Toshiba
- Y1: LCSC Part (none) -> C20625731; MPN (none) -> ABM8-272-T3; Manufacturer (none) -> Abracon
Connections:
- net +3.3V: now also R30.1
- net GND: now also R2.1, J4.1 (EH), J4.2 (EH), J4.3 (EH), J4.4 (EH), J4.A1B12 (GND), J4.B1A12 (GND); no longer R2.2
- net GPIO0: now also R11.2; no longer SW5.1
- net GPIO1: now also U9.5 (VO); no longer SW11.3 (B)
- net GPIO2: now also SW5.1; no longer SW9.3 (B)
- net GPIO3: now also SW11.3 (B); no longer SW10.3 (B)
- net GPIO4: now also SW9.3 (B); no longer SW7.1
- net GPIO5: now also SW10.3 (B)
- net GPIO6: now also SW7.1
- net VBUS: now also J4.A4B9 (VBUS), J4.B4A9 (VBUS)
- net at R5.1, U1.56 (~{QSPI_SS}), U6.1 (~{CS}): now also R30.2
- net at U8.1 (I/O1): now also J4.A7 (DN1), J4.B7 (DN2)
- net at U8.3 (I/O2): now also J4.A6 (DP1), J4.B6 (DP2)
- net at R1.2: now also J4.B5 (CC2)
- new net: J4.A5 (CC1), R2.2
- no-connect marks 38 -> 41
Other:
- moved on the sheet: C14, C7, DS1, R1, R5

Commit message: Lock Hroparts USB-C as J1, qty-5 order carts, and JLCPCB gerbers.
Parts:
- renumbered J4 to J1
Other:
- moved on the sheet: C6, D1, J2, J3, R10, R11, R12, R8, R9, SW10, SW11, SW9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
